File: Boeing/Boeing.kicad_sch (KiCad schematic)
At the start: 0 parts

Commit message: v4 of Boeing SAO
Parts:
- added D: LED, symbol Device:LED
- added J: Conn_02x03_Counter_Clockwise, symbol Connector_Generic:Conn_02x03_Counter_Clockwise
- added R: R, symbol Device:R
Connections:
- new net: D.2 (A), R.1
- new net: J.1 (Pin_1), R.2
- new net: D.1 (K), J.2 (Pin_2)
- no-connect marks 0 -> 4
Changed lines of the file:
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@@
 (kicad_sch (version 20220404) (generator eeschema)
   (paper "A4")
-  (symbol_instances)
+  (no_connect (at 132.08 105.41))
+  (no_connect (at 119.38 110.49))
+  (no_connect (at 132.08 107.95))
+  (no_connect (at 132.08 110.49))
+  (wire (pts (xy 113.03 107.95) (xy 119.38 107.95))
+    (stroke (width 0) (type default))
+  )
+  (wire (pts (xy 119.38 69.85) (xy 124.46 69.85))
+    (stroke (width 0) (type default))
+  )
+  (wire (pts (xy 143.51 119.38) (xy 113.03 119.38))
+    (stroke (width 0) (type default))
+  )
+  (wire (pts (xy 132.08 69.85) (xy 143.51 69.85))
+    (stroke (width 0) (type default))
+  )
+  (wire (pts (xy 143.51 69.85) (xy 143.51 119.38))
+    (stroke (width 0) (type default))
+  )
+  (wire (pts (xy 113.03 119.38) (xy 113.03 107.95))
+    (stroke (width 0) (type default))
+  )
+  (wire (pts (xy 119.38 88.9) (xy 119.38 105.41))
+    (stroke (width 0) (type default))
+  )
+  (wire (pts (xy 119.38 81.28) (xy 119.38 69.85))
+    (stroke (width 0) (type default))
+  )
+  (symbol (lib_id "Device:R") (at 119.38 85.09 0) (unit 1)
+    (in_bom yes) (on_board yes) (fields_autoplaced)
+    (default_instance (reference "R") (unit 1) (value "R") (footprint ""))
+    (property "Reference" "R" (id 0) (at 121.92 84.455 0)
+      (effects (font (size 1.27 1.27)) (justify left))
+    )
+    (property "Value" "R" (id 1) (at 121.92 86.995 0)
+      (effects (font (size 1.27 1.27)) (justify left))
+    )
+    (property "Footprint" "" (id 2) (at 117.602 85.09 90)
+      (effects (font (size 1.27 1.27)) hide)
+    )
+    (property "Datasheet" "~" (id 3) (at 119.38 85.09 0)
+      (effects (font (size 1.27 1.27)) hide)
+    )
+    (pin "1")
+    (pin "2")
+  )
+  (symbol (lib_id "Connector_Generic:Conn_02x03_Counter_Clockwise") (at 124.46 107.95 0) (unit 1)
+    (in_bom yes) (on_board yes) (fields_autoplaced)
+    (default_instance (reference "J") (unit 1) (value "Conn_02x03_Counter_Clockwise") (footprint ""))
+    (property "Reference" "J" (id 0) (at 125.73 100.33 0)
+      (effects (font (size 1.27 1.27)))
+    )
+    (property "Value" "Conn_02x03_Counter_Clockwise" (id 1) (at 125.73 102.87 0)
+      (effects (font (size 1.27 1.27)))
+    )
+    (property "Footprint" "" (id 2) (at 124.46 107.95 0)
+      (effects (font (size 1.27 1.27)) hide)
+    )
+    (property "Datasheet" "~" (id 3) (at 124.46 107.95 0)
+      (effects (font (size 1.27 1.27)) hide)
+    )
+    (pin "1")
+    (pin "2")
+    (pin "3")
+    (pin "4")
+    (pin "5")
+    (pin "6")
+  )
+  (symbol (lib_id "Device:LED") (at 128.27 69.85 180) (unit 1)
+    (in_bom yes) (on_board yes) (fields_autoplaced)
+    (default_instance (reference "D") (unit 1) (value "LED") (footprint ""))
+    (property "Reference" "D" (id 0) (at 129.8575 63.5 0)
+      (effects (font (size 1.27 1.27)))
+    )
+    (property "Value" "LED" (id 1) (at 129.8575 66.04 0)
+      (effects (font (size 1.27 1.27)))
+    )
+    (property "Footprint" "" (id 2) (at 128.27 69.85 0)
+      (effects (font (size 1.27 1.27)) hide)
+    )
+    (property "Datasheet" "~" (id 3) (at 128.27 69.85 0)
+      (effects (font (size 1.27 1.27)) hide)
+    )
+    (pin "1")
+    (pin "2")
+  )
+  (sheet_instances
+    (path "/" (page "1"))
+  )
+  (symbol_instances
+    (path "/bbb6299d-d1fe-454c-a556-8121696b0d88"
+      (reference "D1") (unit 1) (value "LED") (footprint "LED_THT:LED_D5.0mm")
+    )
+    (path "/b071706b-9f82-4349-a4c6-be934fd22e66"
+      (reference "J1") (unit 1) (value "Conn_02x03_Counter_Clockwise") (footprint "Connector_PinHeader_2.54mm:PinHeader_2x03_P2.54mm_Vertical")
+    )
+    (path "/12450330-a01a-4ad9-b262-57aa2d955faa"
+      (reference "R1") (unit 1) (value "R") (footprint "Resistor_SMD:R_1206_3216Metric_Pad1.30x1.75mm_HandSolder")
+    )
+  )
 )
