File: PTP/PTP.kicad_pcb (KiCad board)
At the start: 2 copper layers, 86.5 x 23.9 mm, 3 parts, among them J1 Conn_02x03_Counter_Clockwise

Commit message: v2 of PTP SAO. Attempted to have the non capitalized letters just show as copper
Other:
- board text added: "@av_pubs v2"
- board text removed: "@av_pubs v1"
