File: DDS/DDS.kicad_pcb (KiCad board)
At the start: 0 parts

Commit message: DDS SAO v1
Parts:
- added D1: LED, LED_THT:LED_D5.0mm, F.Cu at (139.7, 114.0)
- added J1: Conn_02x03_Counter_Clockwise, Connector_PinHeader_2.54mm:PinHeader_2x03_P2.54mm_Vertical, B.Cu at (137.2, 99.7)
- added R1: R, Resistor_SMD:R_1206_3216Metric_Pad1.30x1.75mm_HandSolder, B.Cu at (138.4, 107.2)
Routing:
- net Net-(D1-K): track 0.00 -> 25.0 mm
- net Net-(J1-Pin_1): track 0.00 -> 11.1 mm
- net Net-(D1-A): track 0.00 -> 4.43 mm
- added copper zone on B.Cu, net (none)
- added copper zone on F.Cu, net (none)
Other:
- board outline added: 35.5 x 30.5 mm
- copper layers 0 -> 2
- board text added: "@DC30"
- board text added: "@av_pubs v1"
- board text added: "jlcjlcjlcjlc"
