File: AWS/AWS.kicad_pcb (KiCad board)
At the start: 2 copper layers, 75 x 25 mm, 3 parts, among them J1 Conn_02x03_Counter_Clockwise

Commit message: AWS SAO v2
Other:
- board text added: "@av_pubs v2"
- board text removed: "@av_pubs v1"
