File: United/United.kicad_pcb (KiCad board)
At the start: 2 copper layers, 75 x 25 mm, 4 parts, among them J1 Conn_02x03_Counter_Clockwise

Commit message: v2 of United SAO
Parts:
- removed G***: LOGO, LOGO
Other:
- board text added: "@av_pubs v2"
- board text removed: "@DC30"
- board text removed: "@av_pubs v1"
