File: Intelligenesis/IG.kicad_pcb (KiCad board)
At the start: 2 copper layers, 75 x 25 mm, 3 parts, among them J1 Conn_02x03_Counter_Clockwise

Commit message: v2 of Intelligenesis SAO
Parts:
- moved J1 119.5 mm to (218.5, 100.8)
- moved D1 113.9 mm to (221.3, 44.5), turned to 90 degrees
- moved R1 102.3 mm to (204.0, 59.4), turned to 180 degrees
Routing:
- net Net-(D1-K): track 24.1 -> 77.4 mm
- net Net-(J1-Pin_1): track 5.88 -> 48.1 mm
- net Net-(D1-A): track 5.34 -> 24.0 mm
Other:
- board size 75 x 25 mm -> 82.3 x 71.4 mm
- board text added: "@av_pubs v2"
- board text removed: "@av_pubs v1"
