File: Blue Origin/Blue Origin.kicad_pcb (KiCad board)
At the start: 2 copper layers, 70.8 x 28.7 mm, 3 parts, among them J1 Conn_02x03_Counter_Clockwise

Commit message: v3 Blue Origin SAO
Parts:
- moved D1 57.9 mm to (85.1, 113.5), turned to 90 degrees
- moved J1 38.5 mm to (82.7, 102.0)
- moved R1 38.0 mm to (85.3, 96.8), turned to 180 degrees
Routing:
- net Net-(D1-K): track 25.8 -> 9.92 mm
- net Net-(D1-A): track 4.73 -> 16.6 mm
Other:
- board size 70.8 x 28.7 mm -> 12.2 x 86.4 mm
- board text added: "@av_pubs v3"
- board text added: "AV@DC30"
- board text removed: "@av_pubs v2"
